File: mcu.kicad_sch (KiCad schematic)
At the start: 18 parts, among them J1 ARM_JTAG_SWD_10_COMB, U1 PIC32CZ8110CA90208-I/8MX-SL3, Y1 12MHz

Commit message: New design; reduce MCU pin count; utilize new connectors
Parts:
- removed unit 4 of U1
- added D1, D2, D3: H5VL10B, Diode_SMD:D_SOD-882D, symbol Device:D_TVS_Small_Filled
- added J1: USB_C_Receptacle_USB2.0_16P, Connector_USB:USB_C_Receptacle_GCT_USB4105-xx-A_16P_TopMnt_Horizontal, symbol Connector:USB_C_Receptacle_USB2.0_16P
- added R1, R2: 5.1kΩ, Capacitor_SMD:C_0201_0603Metric, symbol Device:R
- D4: renamed from D1; Forward Current 20mA -> (none); Forward Voltage 2V -> (none); JLCPCB Part # C965790 -> C130719; Manufacturer Part # XL-1005SURC -> NCD0402R1
- D7: renamed from D4; JLCPCB Part # C130724 -> C22355736; Manufacturer Part # NCD0402B1 -> XL-1005UBC
- U1: footprint TFBGA208_8MX_MCH -> ul_PIC32CZ8110CA90208-I-8MX-SL3:TFBGA208_8MX_MCH
- renumbered C3 to C2, D2 to D5, D3 to D6, J1 to J2, R7 to R10, R8 to R11, R9 to R3, R10 to R4, R4 to R5, R11 to R6, R12 to R7, R5 to R8, R6 to R9
Connections:
- net GND: now also D1.1 (A1), D2.1 (A1), D3.1 (A1), J1.A1 (GND), J1.A12 (GND), J1.B1 (GND), J1.B12 (GND), R1.2, R2.2
- net VBUS: now also D1.2 (A2), J1.A4 (VBUS), J1.A9 (VBUS), J1.B4 (VBUS), J1.B9 (VBUS)
- new net USB_CC1: J1.A5 (CC1), R2.1
- new net USB_CC2: J1.B5 (CC2), R1.1
- new net USB_D_N: D2.2 (A2), J1.A7 (D-), J1.B7 (D-)
- new net USB_D_P: D3.2 (A2), J1.A6 (D+), J1.B6 (D+)
- no-connect marks 4 -> 7
Other:
- added sheet Power (power.kicad_sch)
- sheet Signal Panel Connectors ports: added CRN_IN_1, CRN_IN_2, CRN_IN_3, CRN_IN_4, CRN_IN_5, CRN_IN_6, CRN_OUT_1, CRN_OUT_2, CRN_OUT_3, CRN_OUT_4, CRN_OUT_5, CRN_OUT_6, SIG_COMP_55, SIG_COMP_56, SIG_OUT_P55, SIG_OUT_P56; removed SIG_OUT_N1, SIG_OUT_N10, SIG_OUT_N11, SIG_OUT_N12, SIG_OUT_N13, SIG_OUT_N14, SIG_OUT_N15, SIG_OUT_N16, SIG_OUT_N17, SIG_OUT_N18, SIG_OUT_N19, SIG_OUT_N2, SIG_OUT_N20, SIG_OUT_N21, SIG_OUT_N22, SIG_OUT_N23, SIG_OUT_N24, SIG_OUT_N25, SIG_OUT_N26, SIG_OUT_N27, SIG_OUT_N28, SIG_OUT_N29, SIG_OUT_N3, SIG_OUT_N30, SIG_OUT_N31, SIG_OUT_N32, SIG_OUT_N33, SIG_OUT_N34, SIG_OUT_N35, SIG_OUT_N36, SIG_OUT_N37, SIG_OUT_N38, SIG_OUT_N39, SIG_OUT_N4, SIG_OUT_N40, SIG_OUT_N41, SIG_OUT_N42, SIG_OUT_N43, SIG_OUT_N44, SIG_OUT_N45, SIG_OUT_N46, SIG_OUT_N47, SIG_OUT_N48, SIG_OUT_N49, SIG_OUT_N5, SIG_OUT_N50, SIG_OUT_N51, SIG_OUT_N52, SIG_OUT_N53, SIG_OUT_N54, SIG_OUT_N6, SIG_OUT_N7, SIG_OUT_N8, SIG_OUT_N9
- note removed: "TODO: Replace Blue LED"
- note removed: "TODO: Replace Red LED"
- moved on the sheet: C1, C2, D4, D5, D6, D7, J2A, R10, R11, R3, R4, R5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

Commit message: Cerberus complete.
Parts:
- added C29: 100nF, Capacitor_SMD:C_0201_0603Metric, symbol Device:C
- added J36: Conn_01x03, Connector_PinHeader_1.27mm:PinHeader_1x03_P1.27mm_Vertical, symbol Connector_Generic:Conn_01x03
- added R232, R234: 10kΩ, Capacitor_SMD:C_0201_0603Metric, symbol Device:R
- added R233: 1kΩ, Capacitor_SMD:C_0201_0603Metric, symbol Device:R
- added SW1, SW2: SW_Push, footprints:YTSB001A0351803B, symbol Switch:SW_Push
Connections:
- net PA7_GPIO_LED_YELLOW is gone; now on net PA29_LED_YELLOW: R9.1
- net PA9_GPIO_LED_RED is gone; now on net PA05_LED_RED: R8.1
- net PD10_GPIO_LED_GREEN is gone; now on net PC11_LED_GREEN: R10.1
- net PE2_GPIO_LED_BLUE is gone; now on net PC03_LED_BLUE: R11.1
- net +3.3V: now also R232.2, R234.2
- net GND: now also C29.2, J36.1 (Pin_1), SW1.1, SW2.1
- net OSC_N: now also U1.A12 (PD0)
- net OSC_P: now also U1.A11 (PD1)
- net PC17_JTAG_TDI: now also U1.D17 (PC17)
- net PC18_JTAG_TMS_SWD: now also U1.C18 (PC18)
- net PC19_JTAG_TDO: now also U1.C17 (PC19)
- net PC20_JTAG_TCK_SWCLK: now also U1.D14 (PC20)
- net RESET_MCU: now also U1.D18 (*RESET), R233.2
- net USB_D_N: now also U1.B18 (D0-)
- net USB_D_P: now also U1.B17 (D0+)
- net PD14_BUS_EN_14: now reaches U1.A10 (PD14)
- net PD10_BUS_EN_18: now reaches U1.A2 (PD10)
- net PD08_BUS_EN_12: now reaches U1.A3 (PD8)
- net PD06_BUS_EN_6: now reaches U1.A4 (PD6)
- net PD19_BUS_EN_2: now reaches U1.A5 (PD19)
- net PD04_BUS_EN_8: now reaches U1.A6 (PD4)
- net PD16_CORNER_IN_1: now reaches U1.A7 (PD16)
- net PD27_BUS_EN_4: now reaches U1.A8 (PD27)
- net PD03_BUS_EN_10: now reaches U1.A9 (PD3)
- net PD12_BUS_EN_16: now reaches U1.B1 (PD12)
- net PD02_BUS_EN_13: now reaches U1.B10 (PD2)
- net PD11_BUS_EN_17: now reaches U1.B2 (PD11)
- net PD09_BUS_EN_11: now reaches U1.B3 (PD9)
- net PD20_BUS_EN_5: now reaches U1.B4 (PD20)
- net PD05_BUS_EN_1: now reaches U1.B5 (PD5)
- net PD18_BUS_EN_7: now reaches U1.B6 (PD18)
- net PD17_CORNER_OUT_1: now reaches U1.B7 (PD17)
- net PD28_BUS_EN_3: now reaches U1.B8 (PD28)
- net PD26_BUS_EN_9: now reaches U1.B9 (PD26)
- net PD24_SERCOM8_DBG_UART_TX: now reaches U1.D11 (PD24)
- net PD24_SERCOM8_DBG_UART_TX: now also J36.3 (Pin_3)
- net PD25_SERCOM8_DBG_UART_RX: now reaches U1.D5 (PD25)
- net PD25_SERCOM8_DBG_UART_RX: now also J36.2 (Pin_2)
- net PC12_BUS_EN_21: now reaches U1.F18 (PC12)
- net PC28_BUS_EN_22: now reaches U1.G18 (PC28)
- net PE00_BUS_EN_26: now reaches U1.H1 (PE0)
- net PC11_LED_GREEN: now reaches U1.H15 (PC11)
- net PC10_DIFF_OUT_-: now reaches U1.H17 (PC10)
- net PE02_BUS_EN_25: now reaches U1.J1 (PE2)
- net PC25_DIFF_OUT_+: now reaches U1.K17 (PC25)
- net PC26_BUS_EN_27: now reaches U1.K18 (PC26)
- net PC31_BUS_EN_28: now reaches U1.L18 (PC31)
- net PC09_CORNER_OUT_4: now reaches U1.M18 (PC9)
- net PC07_CORNER_IN_4: now reaches U1.N18 (PC7)
- net PC22_CORNER_OUT_5: now reaches U1.P18 (PC22)
- net PC03_LED_BLUE: now reaches U1.R17 (PC3)
- net PC04_CORNER_IN_5: now reaches U1.R18 (PC4)
- net PC01_UI_LED_1: now reaches U1.T17 (PC1)
- net PC02_BUS_EN_29: now reaches U1.T18 (PC2)
- net PF04_UI_BUTTON_1: now reaches U1.U10 (PF4)
- net PF00_UI_BUTTON_4: now reaches U1.U7 (PF0)
- net PF03_BUS_EN_48: now reaches U1.V11 (PF3)
- net PF05_BUS_EN_47: now reaches U1.V12 (PF5)
- net PG03_DIFF_IN_+: now reaches U1.G17 (PG3)
- net PG02_BUS_EN_19: now reaches U1.H18 (PG2)
- net PG05_DIFF_IN_-: now reaches U1.J17 (PG5)
- net PG00_BUS_EN_20: now reaches U1.J18 (PG0)
- net PA02_BUS_EN_24: now reaches U1.C1 (PA2)
- net PA01_BUS_EN_15: now reaches U1.C2 (PA1)
- net PA04_CORNER_IN_2: now reaches U1.D1 (PA4)
- net PA03_BUS_EN_23: now reaches U1.D2 (PA3)
- net PA06_CORNER_OUT_2: now reaches U1.E1 (PA6)
- net PA05_LED_RED: now reaches U1.E2 (PA5)
- net PA00_USR_BUTTON: now reaches U1.E4 (PA0)
- net PA00_USR_BUTTON: now also R234.1, SW2.2
- net PA21_CORNER_IN_3: now reaches U1.F1 (PA21)
- net PA23_CORNER_OUT_3: now reaches U1.G1 (PA23)
- net PA24_BUS_EN_32: now reaches U1.M1 (PA24)
- net PA26_BUS_EN_31: now reaches U1.N1 (PA26)
- net PA11_BUS_EN_34: now reaches U1.P1 (PA11)
- net PA13_BUS_EN_33: now reaches U1.R1 (PA13)
- net PA28_BUS_EN_40: now reaches U1.T1 (PA28)
- net PA29_LED_YELLOW: now reaches U1.T2 (PA29)
- net PA15_BUS_EN_39: now reaches U1.U1 (PA15)
- net PB30_UI_LED_4: now reaches U1.U14 (PB30)
- net PB24_UI_LED_3: now reaches U1.U15 (PB24)
- net PB13_UI_LED_2: now reaches U1.U16 (PB13)
- net PB15_BUS_EN_35: now reaches U1.U17 (PB15)
- net PB16_BUS_EN_30: now reaches U1.U18 (PB16)
- net PA16_BUS_EN_44: now reaches U1.U2 (PA16)
- net PA18_PWR_SIG_4: now reaches U1.U3 (PA18)
- net PB03_PWR_SIG_3: now reaches U1.U4 (PB3)
- net PB19_PWR_SIG_2: now reaches U1.U5 (PB19)
- net PB04_PWR_SIG_1: now reaches U1.U6 (PB4)
- net PB23_UI_BUTTON_3: now reaches U1.U8 (PB23)
- net PB08_UI_BUTTON_2: now reaches U1.U9 (PB8/SUPC_OUT1)
- net PB27_BUS_EN_51: now reaches U1.V10 (PB27)
- net PB10_BUS_EN_42: now reaches U1.V13 (PB10)
- net PB11_BUS_EN_41: now reaches U1.V14 (PB11)
- net PB31_BUS_EN_38: now reaches U1.V15 (PB31)
- net PB25_BUS_EN_37: now reaches U1.V16 (PB25)
- net PB14_BUS_EN_36: now reaches U1.V17 (PB14)
- net PB18_BUS_EN_43: now reaches U1.V2 (PB18)
- net PA17_BUS_EN_50: now reaches U1.V3 (PA17)
- net PB20_BUS_EN_49: now reaches U1.V4 (PB20)
- net PB05_BUS_EN_46: now reaches U1.V5 (PB5)
- net PB21_BUS_EN_45: now reaches U1.V6 (PB21)
- net PB06_CORNER_IN_6: now reaches U1.V7 (PB6)
- net PB22_CORNER_OUT_6: now reaches U1.V8 (PB22)
- net PB07_BUS_EN_52: now reaches U1.V9 (PB7/SUPC_OUT0)
- new net _RESET_MCU: C29.1, R232.1, R233.1, SW1.2
- no-connect marks 7 -> 73
Other:
- added sheet Connectors (connectors.kicad_sch)
- sheet Signal Panel Connectors ports: added BUS_EN_1, BUS_EN_10, BUS_EN_11, BUS_EN_12, BUS_EN_13, BUS_EN_14, BUS_EN_15, BUS_EN_16, BUS_EN_17, BUS_EN_18, BUS_EN_19, BUS_EN_2, BUS_EN_20, BUS_EN_21, BUS_EN_22, BUS_EN_23, BUS_EN_24, BUS_EN_25, BUS_EN_26, BUS_EN_27, BUS_EN_28, BUS_EN_29, BUS_EN_3, BUS_EN_30, BUS_EN_31, BUS_EN_32, BUS_EN_33, BUS_EN_34, BUS_EN_35, BUS_EN_36, BUS_EN_37, BUS_EN_38, BUS_EN_39, BUS_EN_4, BUS_EN_40, BUS_EN_41, BUS_EN_42, BUS_EN_43, BUS_EN_44, BUS_EN_45, BUS_EN_46, BUS_EN_47, BUS_EN_48, BUS_EN_49, BUS_EN_5, BUS_EN_50, BUS_EN_51, BUS_EN_52, BUS_EN_6, BUS_EN_7, BUS_EN_8, BUS_EN_9, CORNER_IN_1, CORNER_IN_2, CORNER_IN_3, CORNER_IN_4, CORNER_IN_5, CORNER_IN_6, CORNER_OUT_1, CORNER_OUT_2, CORNER_OUT_3, CORNER_OUT_4, CORNER_OUT_5, CORNER_OUT_6, DIFF_IN_+, DIFF_IN_-, DIFF_OUT_+, DIFF_OUT_-; removed CRN_IN_1, CRN_IN_2, CRN_IN_3, CRN_IN_4, CRN_IN_5, CRN_IN_6, CRN_OUT_1, CRN_OUT_2, CRN_OUT_3, CRN_OUT_4, CRN_OUT_5, CRN_OUT_6, SIG_COMP_1, SIG_COMP_10, SIG_COMP_11, SIG_COMP_12, SIG_COMP_13, SIG_COMP_14, SIG_COMP_15, SIG_COMP_16, SIG_COMP_17, SIG_COMP_18, SIG_COMP_19, SIG_COMP_2, SIG_COMP_20, SIG_COMP_21, SIG_COMP_22, SIG_COMP_23, SIG_COMP_24, SIG_COMP_25, SIG_COMP_26, SIG_COMP_27, SIG_COMP_28, SIG_COMP_29, SIG_COMP_3, SIG_COMP_30, SIG_COMP_31, SIG_COMP_32, SIG_COMP_33, SIG_COMP_34, SIG_COMP_35, SIG_COMP_36, SIG_COMP_37, SIG_COMP_38, SIG_COMP_39, SIG_COMP_4, SIG_COMP_40, SIG_COMP_41, SIG_COMP_42, SIG_COMP_43, SIG_COMP_44, SIG_COMP_45, SIG_COMP_46, SIG_COMP_47, SIG_COMP_48, SIG_COMP_49, SIG_COMP_5, SIG_COMP_50, SIG_COMP_51, SIG_COMP_52, SIG_COMP_53, SIG_COMP_54, SIG_COMP_55, SIG_COMP_56, SIG_COMP_6, SIG_COMP_7, SIG_COMP_8, SIG_COMP_9, SIG_OUT_P1, SIG_OUT_P10, SIG_OUT_P11, SIG_OUT_P12, SIG_OUT_P13, SIG_OUT_P14, SIG_OUT_P15, SIG_OUT_P16, SIG_OUT_P17, SIG_OUT_P18, SIG_OUT_P19, SIG_OUT_P2, SIG_OUT_P20, SIG_OUT_P21, SIG_OUT_P22, SIG_OUT_P23, SIG_OUT_P24, SIG_OUT_P25, SIG_OUT_P26, SIG_OUT_P27, SIG_OUT_P28, SIG_OUT_P29, SIG_OUT_P3, SIG_OUT_P30, SIG_OUT_P31, SIG_OUT_P32, SIG_OUT_P33, SIG_OUT_P34, SIG_OUT_P35, SIG_OUT_P36, SIG_OUT_P37, SIG_OUT_P38, SIG_OUT_P39, SIG_OUT_P4, SIG_OUT_P40, SIG_OUT_P41, SIG_OUT_P42, SIG_OUT_P43, SIG_OUT_P44, SIG_OUT_P45, SIG_OUT_P46, SIG_OUT_P47, SIG_OUT_P48, SIG_OUT_P49, SIG_OUT_P5, SIG_OUT_P50, SIG_OUT_P51, SIG_OUT_P52, SIG_OUT_P53, SIG_OUT_P54, SIG_OUT_P55, SIG_OUT_P56, SIG_OUT_P6, SIG_OUT_P7, SIG_OUT_P8, SIG_OUT_P9
- moved on the sheet: C1, C2, D1, D2, D3, D4, D5, D6, D7, J1, J2A, R1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
