File: outer_panel_conn.kicad_sch (KiCad schematic)
At the start: 37 parts, among them J3 Molex_5051101697, U2 SN74LVC125ARGYR, U3 SN74LVC2G04DCKR, U4 LM393LVDSGR

Commit message: Cerberus complete.
Parts:
- removed C10, C11: 100nF, Capacitor_SMD:C_0201_0603Metric, symbol Device:C
- removed C3, C4, C5, C6, C8, C9: 47pF, Capacitor_SMD:C_0201_0603Metric, symbol Device:C
- removed R13, R14, R15, R20, R21: 47Ω, Resistor_SMD:R_0201_0603Metric, symbol Device:R
- removed R16, R17, R18, R19, R22, R23: 10kΩ, Capacitor_SMD:C_0201_0603Metric, symbol Device:R
- removed R24, R25: 680kΩ, Resistor_SMD:R_0201_0603Metric, symbol Device:R
- removed U2: SN74LVC125ARGYR, ul_SN74LVC125ARGYR:RGY14_2P05X2P05, symbol SN74LVC125ARGYR:SN74LVC125ARGYR
- removed U3: SN74LVC2G04DCKR, Package_TO_SOT_SMD:SOT-363_SC-70-6, symbol SN74LVC2G04DCKR:SN74LVC2G04DCKR
- removed U4: LM393LVDSGR, ul_LM393LVDSGR:WSON8_DSG_TEX, symbol LM393LVDSGR:LM393LVDSGR
- added R32, R33, R34, R35, R36, R38, R39, R40, R41: 100Ω, Resistor_SMD:R_0201_0603Metric, symbol Device:R
- added U5: SN74LVC244ARGYR, ul_SN74LVC244ARGYR:RGY20_3P05X2P05, symbol SN74LVC244ARGYR:SN74LVC244ARGYR
- R30: renamed from R12; value 47Ω -> 100Ω; JLCPCB Part # C273279 -> C270366; Manufacturer Part # RC0201FR-0747RL -> 0201WMF1000TEE
- renumbered C7 to C6, D8 to D24, D9 to D25, D10 to D26, D11 to D27, D12 to D28, D13 to D29, D14 to D30, D15 to D31, D16 to D32, D17 to D33, J3 to J5
Connections:
- net +3.3V: now also U5.20 (VCC)
- net CORNER_IN: now also R41.2
- net CORNER_OUT: now also R40.2
- net GND: now also U5.10 (GND), U5.21 (EPAD)
- net CORNER_A_IN renamed CORNER_IN_A
- net CORNER_IN_A: now also R41.1
- net CORNER_A_OUT renamed CORNER_OUT_A
- net CORNER_OUT_A: now also R40.1
- net SIN_B_1_N renamed DIFF_IN_A_1_-
- net DIFF_IN_A_1_-: now also R36.1
- net SIN_B_1_P renamed DIFF_IN_A_1_+
- net DIFF_IN_A_1_+: now also R35.1
- net SIN_B_2_N renamed DIFF_IN_A_2_-
- net DIFF_IN_A_2_-: now also R39.1
- net SIN_B_2_P renamed DIFF_IN_A_2_+
- net DIFF_IN_A_2_+: now also R38.1
- net SOUT_A_1_P renamed DIFF_OUT_1_+
- net DIFF_OUT_1_+: now also U5.18 (1Y1)
- net SOUT_B_1_N renamed DIFF_OUT_A_1_-
- net DIFF_OUT_A_1_-: now also R32.1
- net SOUT_B_1_P renamed DIFF_OUT_A_1_+
- net SOUT_B_2_N renamed DIFF_OUT_A_2_-
- net DIFF_OUT_A_2_-: now also R34.1
- net SOUT_B_2_P renamed DIFF_OUT_A_2_+
- net DIFF_OUT_A_2_+: now also R33.1
- new net BUS_EN_1: U5.1 (*1OE)
- new net BUS_EN_2: U5.19 (*2OE)
- new net DIFF_IN_+: U5.14 (1Y3), U5.5 (2Y3)
- new net DIFF_IN_-: U5.12 (1Y4), U5.3 (2Y4)
- new net DIFF_IN_1_+: R35.2, U5.6 (1A3)
- new net DIFF_IN_1_-: R36.2, U5.8 (1A4)
- new net DIFF_IN_2_+: R38.2, U5.15 (2A3)
- new net DIFF_IN_2_-: R39.2, U5.17 (2A4)
- new net DIFF_OUT_+: U5.11 (2A1), U5.2 (1A1)
- new net DIFF_OUT_-: U5.13 (2A2), U5.4 (1A2)
- new net DIFF_OUT_1_-: R32.2, U5.16 (1Y2)
- new net DIFF_OUT_2_+: R33.2, U5.9 (2Y1)
- new net DIFF_OUT_2_-: R34.2, U5.7 (2Y2)
Other:
- note removed: "Dual Comparator"
- note removed: "Dual Inverter"
- note removed: "Quad Buffer"
- moved on the sheet: C6, D24, D25, D26, D27, D28, D29, D30, D31, D32, D33, J5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
