File: power.kicad_sch (KiCad schematic)
At the start: 35 parts, among them U1 PIC32CZ8110CA90208-I/8MX-SL3, U86 AMS1117-3.3, U87 RT9013-18GB

Commit message: Cerberus complete.
Parts:
- added D220: Schottkey, Diode_SMD:D_SOD-323, symbol Device:D_Schottky_Filled
- added D221: H5VL10B, Diode_SMD:D_SOD-882D, symbol Device:D_TVS_Small_Filled
- added J34: Conn_01x02, Connector_PinHeader_2.54mm:PinHeader_1x02_P2.54mm_Horizontal, symbol Connector_Generic:Conn_01x02
Connections:
- net +3.3V: now also U1.B16 (VUSB3VB3_0); no longer U1.B13 (VUSB3V3_1)
- net GND: now also D221.2 (A2), J34.2 (Pin_2)
- net VDD: now also D220.1 (K)
- net VIN: now also D221.1 (A1), J34.1 (Pin_1)
- new net VAA: D220.2 (A)
Other:
- moved on the sheet: C267, C271, C272, C280, C281, C282, D244, D245, U86, U87
