File: connectors.kicad_sch (KiCad schematic)
At the start: 32 parts, among them J32 Molex_5051101697, J33 Molex_5051101292

Commit message: fab outputs, full 3D model, and minor improvements
Parts:
- J33: JLCPCB Part # (none) -> C585301; Manufacturer Part # (none) -> 5051101292; Status (none) -> Extended
Changed lines of the file:
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@@
 			)
 		)
-		(property "JLCPCB Part #" "~"
+		(property "JLCPCB Part #" "C585301"
 			(at 67.31 132.08 0)
 			(effects
@@
 			)
 		)
-		(property "Manufacturer Part #" "~"
+		(property "Manufacturer Part #" "5051101292"
 			(at 67.31 132.08 0)
 			(effects
@@
 			)
 		)
-		(property "Status" "~"
+		(property "Status" "Extended"
 			(at 67.31 132.08 0)
 			(effects
