File: d_inner_sml_panel_conn.kicad_sch (KiCad schematic)
At the start: 34 parts, among them J10 Molex_5051100692, J11 Molex_5051100692, U23 SN74LVC125ARGYR, U24 SN74LVC2G04DCKR, U25 LM393LVDSGR

Commit message: Cerberus complete.
Parts:
- removed C66, C67, C68, C69, C71, C72: 47pF, Capacitor_SMD:C_0201_0603Metric, symbol Device:C
- removed C70, C73, C74: 100nF, Capacitor_SMD:C_0201_0603Metric, symbol Device:C
- removed R116, R117: 10kΩ, Capacitor_SMD:C_0201_0603Metric, symbol Device:R
- removed R118, R119: 680kΩ, Resistor_SMD:R_0201_0603Metric, symbol Device:R
- removed U23: SN74LVC125ARGYR, ul_SN74LVC125ARGYR:RGY14_2P05X2P05, symbol SN74LVC125ARGYR:SN74LVC125ARGYR
- removed U24: SN74LVC2G04DCKR, Package_TO_SOT_SMD:SOT-363_SC-70-6, symbol SN74LVC2G04DCKR:SN74LVC2G04DCKR
- removed U25: LM393LVDSGR, ul_LM393LVDSGR:WSON8_DSG_TEX, symbol LM393LVDSGR:LM393LVDSGR
- added C22: 100nF, Capacitor_SMD:C_0201_0603Metric, symbol Device:C
- added U20: SN74LVC244ARGYR, ul_SN74LVC244ARGYR:RGY20_3P05X2P05, symbol SN74LVC244ARGYR:SN74LVC244ARGYR
- R108, R109, R110, R111: value 47Ω -> 100Ω; JLCPCB Part # C273279 -> C270366; Manufacturer Part # RC0201FR-0747RL -> 0201WMF1000TEE
- R112, R113, R114, R115: value 10kΩ -> 100Ω; footprint Capacitor_SMD:C_0201_0603Metric -> Resistor_SMD:R_0201_0603Metric; JLCPCB Part # C106225 -> C270366; Manufacturer Part # RC0201FR-0710KL -> 0201WMF1000TEE
Connections:
- net +3.3V: now also C22.2, U20.20 (VCC)
- net GND: now also C22.1, U20.10 (GND), U20.21 (EPAD)
- net SIN_A_1_N renamed DIFF_IN_A_1_-
- net DIFF_IN_A_1_-: now also D81.1 (A1), J10.6 (Pin_6)
- net SIN_A_1_P renamed DIFF_IN_A_1_+
- net DIFF_IN_A_1_+: now also D80.1 (A1), J10.5 (Pin_5)
- net SIN_A_2_N renamed DIFF_IN_A_2_-
- net DIFF_IN_A_2_-: now also D83.1 (A1), J11.6 (Pin_6)
- net SIN_A_2_P renamed DIFF_IN_A_2_+
- net DIFF_IN_A_2_+: now also D82.1 (A1), J11.5 (Pin_5)
- removed net SIN_B_1_N: D81.1 (A1), J10.6 (Pin_6), R113.2
- removed net SIN_B_1_P: D80.1 (A1), J10.5 (Pin_5), R112.2
- removed net SIN_B_2_N: D83.1 (A1), J11.6 (Pin_6), R115.2
- removed net SIN_B_2_P: D82.1 (A1), J11.5 (Pin_5), R114.2
- net SOUT_A_1_N renamed DIFF_OUT_1_-
- net DIFF_OUT_1_-: now also U20.16 (1Y2)
- net SOUT_A_1_P renamed DIFF_OUT_1_+
- net DIFF_OUT_1_+: now also U20.18 (1Y1)
- net SOUT_A_2_N renamed DIFF_OUT_2_-
- net DIFF_OUT_2_-: now also U20.7 (2Y2)
- net SOUT_A_2_P renamed DIFF_OUT_2_+
- net DIFF_OUT_2_+: now also U20.9 (2Y1)
- net SOUT_B_1_N renamed DIFF_OUT_A_1_-
- net SOUT_B_1_P renamed DIFF_OUT_A_1_+
- net SOUT_B_2_N renamed DIFF_OUT_A_2_-
- net SOUT_B_2_P renamed DIFF_OUT_A_2_+
- new net BUS_EN_1: U20.1 (*1OE)
- new net BUS_EN_2: U20.19 (*2OE)
- new net DIFF_IN_+: U20.14 (1Y3), U20.5 (2Y3)
- new net DIFF_IN_-: U20.12 (1Y4), U20.3 (2Y4)
- new net DIFF_IN_1_+: R112.2, U20.6 (1A3)
- new net DIFF_IN_1_-: R113.2, U20.8 (1A4)
- new net DIFF_IN_2_+: R114.2, U20.15 (2A3)
- new net DIFF_IN_2_-: R115.2, U20.17 (2A4)
- new net DIFF_OUT_+: U20.11 (2A1), U20.2 (1A1)
- new net DIFF_OUT_-: U20.13 (2A2), U20.4 (1A2)
Other:
- note removed: "Dual Comparator"
- note removed: "Dual Inverter"
- note removed: "Quad Buffer"
- moved on the sheet: D76, D77, D78, D79, D80, D81, D82, J10, J11

Commit message: fab outputs, full 3D model, and minor improvements
Parts:
- J10, J11: JLCPCB Part # (none) -> C779386; Manufacturer Part # (none) -> 5051100692; Status (none) -> Extended
