File: inner_panel_conn.kicad_sch (KiCad schematic)
At the start: 33 parts, among them J9 Molex_5051101292, U20 SN74LVC125ARGYR, U21 SN74LVC2G04DCKR, U22 LM393LVDSGR

Commit message: Cerberus complete.
Parts:
- removed C57, C58, C59, C60, C62, C63: 47pF, Capacitor_SMD:C_0201_0603Metric, symbol Device:C
- removed C61, C64, C65: 100nF, Capacitor_SMD:C_0201_0603Metric, symbol Device:C
- removed D68, D69, D70, D71, D72, D73, D74, D75: H5VL10B, Diode_SMD:D_SOD-882D, symbol Device:D_TVS_Small_Filled
- removed J9: Molex_5051101292, ul_5051101292:CON_5051101292_MOL, symbol Connector_Generic:Conn_01x12
- removed R100, R101, R102, R103, R104, R105: 10kΩ, Capacitor_SMD:C_0201_0603Metric, symbol Device:R
- removed R106, R107: 680kΩ, Resistor_SMD:R_0201_0603Metric, symbol Device:R
- removed R96, R97, R98, R99: 47Ω, Resistor_SMD:R_0201_0603Metric, symbol Device:R
- removed U20: SN74LVC125ARGYR, ul_SN74LVC125ARGYR:RGY14_2P05X2P05, symbol SN74LVC125ARGYR:SN74LVC125ARGYR
- removed U21: SN74LVC2G04DCKR, Package_TO_SOT_SMD:SOT-363_SC-70-6, symbol SN74LVC2G04DCKR:SN74LVC2G04DCKR
- removed U22: LM393LVDSGR, ul_LM393LVDSGR:WSON8_DSG_TEX, symbol LM393LVDSGR:LM393LVDSGR
- added C4: 100nF, Capacitor_SMD:C_0201_0603Metric, symbol Device:C
- added D10, D11, D12, D13, D14, D15, D8, D9: H5VL10B, Diode_SMD:D_SOD-882D, symbol Device:D_TVS_Small_Filled
- added J3: Molex_5051101292, ul_5051101292:CON_5051101292_MOL, symbol Connector_Generic:Conn_01x12
- added R12, R13, R14, R15, R16, R17, R19, R20: 100Ω, Resistor_SMD:R_0201_0603Metric, symbol Device:R
- added U3: SN74LVC244ARGYR, ul_SN74LVC244ARGYR:RGY20_3P05X2P05, symbol SN74LVC244ARGYR:SN74LVC244ARGYR
Connections:
- net +3.3V: now also C4.2, U3.20 (VCC)
- net GND: now also C4.1, D10.2 (A2), D11.2 (A2), D12.2 (A2), D13.2 (A2), D14.2 (A2), D15.2 (A2), D8.2 (A2), D9.2 (A2), J3.1 (Pin_1), J3.10 (Pin_10), J3.4 (Pin_4), J3.7 (Pin_7), U3.10 (GND), U3.21 (EPAD)
- new net BUS_EN_1: U3.1 (*1OE)
- new net BUS_EN_2: U3.19 (*2OE)
- new net DIFF_IN_+: U3.14 (1Y3), U3.5 (2Y3)
- new net DIFF_IN_-: U3.12 (1Y4), U3.3 (2Y4)
- new net DIFF_IN_1_+: R16.2, U3.6 (1A3)
- new net DIFF_IN_1_-: R17.2, U3.8 (1A4)
- new net DIFF_IN_2_+: R19.2, U3.15 (2A3)
- new net DIFF_IN_2_-: R20.2, U3.17 (2A4)
- new net DIFF_IN_A_1_+: D12.1 (A1), J3.8 (Pin_8), R16.1
- new net DIFF_IN_A_1_-: D13.1 (A1), J3.9 (Pin_9), R17.1
- new net DIFF_IN_A_2_+: D14.1 (A1), J3.11 (Pin_11), R19.1
- new net DIFF_IN_A_2_-: D15.1 (A1), J3.12 (Pin_12), R20.1
- new net DIFF_OUT_+: U3.11 (2A1), U3.2 (1A1)
- new net DIFF_OUT_-: U3.13 (2A2), U3.4 (1A2)
- new net DIFF_OUT_1_+: R12.2, U3.18 (1Y1)
- new net DIFF_OUT_1_-: R13.2, U3.16 (1Y2)
- new net DIFF_OUT_2_+: R14.2, U3.9 (2Y1)
- new net DIFF_OUT_2_-: R15.2, U3.7 (2Y2)
- new net DIFF_OUT_A_1_+: D8.1 (A1), J3.2 (Pin_2), R12.1
- new net DIFF_OUT_A_1_-: D9.1 (A1), J3.3 (Pin_3), R13.1
- new net DIFF_OUT_A_2_+: D10.1 (A1), J3.5 (Pin_5), R14.1
- new net DIFF_OUT_A_2_-: D11.1 (A1), J3.6 (Pin_6), R15.1
Other:
- note removed: "Dual Comparator"
- note removed: "Dual Inverter"
- note removed: "Quad Buffer"

Commit message: fab outputs, full 3D model, and minor improvements
Parts:
- J3: JLCPCB Part # (none) -> C585301; Manufacturer Part # (none) -> 5051101292; Status (none) -> Extended
Changed lines of the file:
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@@
 			)
 		)
-		(property "JLCPCB Part #" "~"
+		(property "JLCPCB Part #" "C585301"
 			(at 29.21 88.9 0)
 			(effects
@@
 			)
 		)
-		(property "Manufacturer Part #" "~"
+		(property "Manufacturer Part #" "5051101292"
 			(at 29.21 88.9 0)
 			(effects
@@
 			)
 		)
-		(property "Status" "~"
+		(property "Status" "Extended"
 			(at 29.21 88.9 0)
 			(effects
